Commit message: train

File: roboverse_pack/robots_vega/humanoid/vega_1/vega.urdf (robot description, URDF)
Before this commit: robot vega-1, 79 links, 78 joints
Links:
- removed link head_l1
- removed link head_l2
- removed link head_l3
- link arm_center: mass 0.001 -> 1.6793; geometry collision mesh filename=meshes/collision/head_l1.obj; collision mesh filename=meshes/collision/head_l2.obj
Joints:
- removed joint head_j1
- removed joint head_j2
- removed joint head_j3
- joint zed_left_camera_mount: origin xyz=0.0365 0.023 0.0489 rpy=-1.57079 0 -1.57079 -> xyz=-0.037 0.025 0.1089 rpy=-1.57079 0 -1.57079; parent head_l3 -> arm_center
- joint zed_left_depth_mount: origin xyz=0.025 0.023 0.0489 rpy=-1.57079 0 -1.57079 -> xyz=-0.0485 0.025 0.1089 rpy=-1.57079 0 -1.57079; parent head_l3 -> arm_center
- joint zed_right_camera_mount: origin xyz=0.0365 -0.027 0.0489 rpy=-1.57079 0 -1.57079 -> xyz=-0.037 -0.025 0.1089 rpy=-1.57079 0 -1.57079; parent head_l3 -> arm_center

File: roboverse_pack/whale_doll.urdf (robot description, URDF)
Before this commit: robot whale_doll, 1 links, 0 joints
Links:
- link whale_doll: mass 0.800000 -> 0.050000; geometry collision mesh filename=collision_meshes/whale_doll_convex_00.obj; collision mesh filename=collision_meshes/whale_doll_convex_01.obj

Commit message: fix urdf & usd

File: roboverse_pack/robots_vega/humanoid/vega_1/vega.urdf (robot description, URDF)
Before this commit: robot vega-1, 76 links, 75 joints
Joints:
- joint R_ff_j1: axis 0 1 0 -> (none); limit lower=-1.0946 upper=0.2891 effort=0.5 velocity=6.28 -> (none); type revolute -> fixed
- joint R_ff_j2: axis 0 1 0 -> (none); limit lower=-1.2101 upper=0.3681 effort=0.5 velocity=6.28 -> (none); mimic joint=R_ff_j1 multiplier=1.13028 offset=-0.00053 -> (none); type revolute -> fixed
- joint R_lf_j1: axis 0 1 0 -> (none); limit lower=-1.0118 upper=0.2811 effort=0.5 velocity=6.28 -> (none); type revolute -> fixed
- joint R_lf_j2: axis 0 1 0 -> (none); limit lower=-1.1073 upper=0.4014 effort=0.5 velocity=6.28 -> (none); mimic joint=R_lf_j1 multiplier=1.15037 offset=0.00186 -> (none); type revolute -> fixed
- joint R_mf_j1: axis 0 1 0 -> (none); limit lower=-1.0844 upper=0.2801 effort=0.5 velocity=6.28 -> (none); type revolute -> fixed
- joint R_mf_j2: axis 0 1 0 -> (none); limit lower=-1.2026 upper=0.3533 effort=0.5 velocity=6.28 -> (none); mimic joint=R_mf_j1 multiplier=1.13311 offset=-0.00079 -> (none); type revolute -> fixed
- joint R_rf_j1: axis 0 1 0 -> (none); limit lower=-1.0154 upper=0.2840 effort=0.5 velocity=6.28 -> (none); type revolute -> fixed
- joint R_rf_j2: axis 0 1 0 -> (none); limit lower=-1.1156 upper=0.3599 effort=0.5 velocity=6.28 -> (none); mimic joint=R_rf_j1 multiplier=1.12935 offset=0.00065 -> (none); type revolute -> fixed
- joint R_th_j0: axis 1 0 0 -> (none); limit lower=-0.0158 upper=1.605 effort=1.0 velocity=6.28 -> (none); type revolute -> fixed
- joint R_th_j1: axis 0 0 -1 -> (none); limit lower=-0.3468 upper=0.1834 effort=1.0 velocity=6.28 -> (none); type revolute -> fixed
- joint R_th_j2: axis 0 0 -1 -> (none); limit lower=-0.4298 upper=0.2731 effort=0.5 velocity=6.28 -> (none); mimic joint=R_th_j1 multiplier=1.35316 offset=0.00765 -> (none); type revolute -> fixed
